File: schematics/sensor_pcb/sensor_pcb.kicad_pcb (KiCad board)
At the start: 2 copper layers, 28 x 32 mm, 21 parts, among them J1 Conn_01x08, U1 PMW3360DM-T2QU, U2 TLV74318PDBVR

Commit message: Update
Parts:
- moved C5 0.18 mm to (226.2, 141.1)
- moved U2 0.18 mm to (219.8, 140.1)
- moved C3 0.18 mm to (216.5, 140.1)
- moved C4 0.18 mm to (223.1, 140.1)
- moved R4 0.18 mm to (226.2, 139.1)
Routing:
- net GND: track 4.83 -> 16.6 mm, vias 0 -> 2
- net VDD: track 41.7 -> 39.3 mm
- net Net-(U2-NC): track 8.77 -> 10.6 mm
